Commit message: Add five-axis stator-mounted press tool model

File: src/piper_description/urdf/piper_description.xacro (robot description, xacro)
@@ -3,5 +3,7 @@
   name="piper"
   xmlns:xacro="http://ros.org/wiki/xacro">
+  <xacro:arg name="use_press_tool" default="false" />
   <xacro:include filename="$(find piper_description)/urdf/wrist_depth_camera.xacro" />
+  <xacro:include filename="$(find piper_description)/urdf/piper_press_tool.xacro" />
 <!-- world -->
   <link name="world"/>
@@ -320,22 +322,23 @@
     </collision>
   </link>
-  <joint
-    name="joint6"
-    type="revolute">
-    <origin
-      xyz="8.8259E-05 -0.091 0"
-      rpy="1.5708 0 0" />
-    <parent
-      link="link5" />
-    <child
-      link="link6" />
-    <axis
-      xyz="0 0 1" />
-    <limit
-      lower="-2.0944"
-      upper="2.0944"
-      effort="100"
-      velocity="3" />
-  </joint>
+  <xacro:unless value="$(arg use_press_tool)">
+    <joint name="joint6" type="revolute">
+      <origin xyz="8.8259E-05 -0.091 0" rpy="1.5708 0 0" />
+      <parent link="link5" />
+      <child link="link6" />
+      <axis xyz="0 0 1" />
+      <limit lower="-2.0944" upper="2.0944" effort="100" velocity="3" />
+    </joint>
+  </xacro:unless>
+  <xacro:if value="$(arg use_press_tool)">
+    <!-- The unused rotor is retained at its zero pose for collision geometry. -->
+    <joint name="joint6_fixed" type="fixed">
+      <origin xyz="8.8259E-05 -0.091 0" rpy="1.5708 0 0" />
+      <parent link="link5" />
+      <child link="link6" />
+    </joint>
+    <xacro:piper_press_tool parent_link="link5" enable_gazebo="false" />
+  </xacro:if>
+  <xacro:unless value="$(arg use_press_tool)">
   <link
     name="gripper_base">
@@ -506,4 +509,5 @@
       velocity="1" />
   </joint>
+  </xacro:unless>
 <!-- controller -->
   <xacro:macro name="transmission_block" params="tran_name joint_name motor_name">
@@ -524,7 +528,9 @@
   <xacro:transmission_block tran_name="tran4" joint_name="joint4" motor_name="motor4"/>
   <xacro:transmission_block tran_name="tran5" joint_name="joint5" motor_name="motor5"/>
-  <xacro:transmission_block tran_name="tran6" joint_name="joint6" motor_name="motor6"/>
-  <xacro:transmission_block tran_name="tran7" joint_name="joint7" motor_name="motor7"/>
-  <xacro:transmission_block tran_name="tran8" joint_name="joint8" motor_name="motor8"/>
+  <xacro:unless value="$(arg use_press_tool)">
+    <xacro:transmission_block tran_name="tran6" joint_name="joint6" motor_name="motor6"/>
+    <xacro:transmission_block tran_name="tran7" joint_name="joint7" motor_name="motor7"/>
+    <xacro:transmission_block tran_name="tran8" joint_name="joint8" motor_name="motor8"/>
+  </xacro:unless>
 <!-- gazebo -->
   <gazebo>

File: src/piper_description/urdf/piper_description_gazebo.xacro (robot description, xacro)
@@ -3,5 +3,7 @@
   name="piper"
   xmlns:xacro="http://ros.org/wiki/xacro">
+  <xacro:arg name="use_press_tool" default="false" />
   <xacro:include filename="$(find piper_description)/urdf/wrist_depth_camera.xacro" />
+  <xacro:include filename="$(find piper_description)/urdf/piper_press_tool.xacro" />
 <!-- world -->
   <link name="world"/>
@@ -320,22 +322,22 @@
     </collision>
   </link>
-  <joint
-    name="joint6"
-    type="revolute">
-    <origin
-      xyz="8.8259E-05 -0.091 0"
-      rpy="1.5708 0 0" />
-    <parent
-      link="link5" />
-    <child
-      link="link6" />
-    <axis
-      xyz="0 0 1" />
-    <limit
-      lower="-2.0944"
-      upper="2.0944"
-      effort="100"
-      velocity="3" />
-  </joint>
+  <xacro:unless value="$(arg use_press_tool)">
+    <joint name="joint6" type="revolute">
+      <origin xyz="8.8259E-05 -0.091 0" rpy="1.5708 0 0" />
+      <parent link="link5" />
+      <child link="link6" />
+      <axis xyz="0 0 1" />
+      <limit lower="-2.0944" upper="2.0944" effort="100" velocity="3" />
+    </joint>
+  </xacro:unless>
+  <xacro:if value="$(arg use_press_tool)">
+    <joint name="joint6_fixed" type="fixed">
+      <origin xyz="8.8259E-05 -0.091 0" rpy="1.5708 0 0" />
+      <parent link="link5" />
+      <child link="link6" />
+    </joint>
+    <xacro:piper_press_tool parent_link="link5" enable_gazebo="true" />
+  </xacro:if>
+  <xacro:unless value="$(arg use_press_tool)">
   <link
     name="gripper_base">
@@ -506,4 +508,5 @@
       velocity="1" />
   </joint>
+  </xacro:unless>
   <!-- <gazebo reference="base_link">
       <material>Gazebo/Black</material>
@@ -591,39 +594,46 @@
           <state_interface name="velocity"/>
       </joint>
-      <joint name="joint6">
-          <command_interface name="position">
-              <param name="min">-1</param>
-              <param name="max">1</param>
-          </command_interface>
-          <state_interface name="position">
-              <param name="initial_value">0.0</param>
-          </state_interface>
-          <state_interface name="velocity"/>
-      </joint>
-      <joint name="joint7">
-          <command_interface name="position">
-              <param name="min">-1</param>
-              <param name="max">1</param>
-          </command_interface>
-          <state_interface name="position">
-              <param name="initial_value">0.0</param>
-          </state_interface>
-          <state_interface name="velocity"/>
-      </joint>
-      <joint name="joint8">
-          <command_interface name="position">
-              <param name="min">-1</param>
-              <param name="max">1</param>
-          </command_interface>
-          <state_interface name="position">
-              <param name="initial_value">0.0</param>
-          </state_interface>
-          <state_interface name="velocity"/>
-      </joint>
+      <xacro:unless value="$(arg use_press_tool)">
+        <joint name="joint6">
+            <command_interface name="position">
+                <param name="min">-1</param>
+                <param name="max">1</param>
+            </command_interface>
+            <state_interface name="position">
+                <param name="initial_value">0.0</param>
+            </state_interface>
+            <state_interface name="velocity"/>
+        </joint>
+        <joint name="joint7">
+            <command_interface name="position">
+                <param name="min">-1</param>
+                <param name="max">1</param>
+            </command_interface>
+            <state_interface name="position">
+                <param name="initial_value">0.0</param>
+            </state_interface>
+            <state_interface name="velocity"/>
+        </joint>
+        <joint name="joint8">
+            <command_interface name="position">
+                <param name="min">-1</param>
+                <param name="max">1</param>
+            </command_interface>
+            <state_interface name="position">
+                <param name="initial_value">0.0</param>
+            </state_interface>
+            <state_interface name="velocity"/>
+        </joint>
+      </xacro:unless>
   </ros2_control>
 <!-- gazebo -->
   <gazebo>
     <plugin name="gazebo_ros2_control" filename="libgazebo_ros2_control.so">
-        <parameters> $(find piper_gazebo)/config/ros2_controllers.yaml </parameters>
+        <xacro:if value="$(arg use_press_tool)">
+          <parameters>$(find piper_gazebo)/config/press_ros2_controllers.yaml</parameters>
+        </xacro:if>
+        <xacro:unless value="$(arg use_press_tool)">
+          <parameters>$(find piper_gazebo)/config/ros2_controllers.yaml</parameters>
+        </xacro:unless>
         <robot_param_node>robot_state_publisher</robot_param_node>
     </plugin>
